File: robomow_city120_terminal.sch (EAGLE design)
At the start: 10 parts, among them J1 RJ11-2L-B

Commit message: Added logs, revenged terminal commands
Connections:
- net N$1 renamed TX_R
- net N$2 renamed RX_R
Changed lines of the file:
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@@
 <?xml version="1.0" encoding="utf-8"?>
 <!DOCTYPE eagle SYSTEM "eagle.dtd">
-<eagle version="9.3.0">
+<eagle version="9.4.2">
 <drawing>
 <settings>
@@
 </segment>
 </net>
-<net name="N$1" class="0">
+<net name="TX_R" class="0">
 <segment>
 <pinref part="R1" gate="G$1" pin="1"/>
@@
 </segment>
 </net>
-<net name="N$2" class="0">
+<net name="RX_R" class="0">
 <segment>
 <pinref part="R2" gate="G$1" pin="1"/>
