File: DualFlash adapter/dual flash adapter.kicad_pcb (KiCad board)
At the start: 2 copper layers, 55 x 25 mm, 11 parts, among them IC1 SN74LVC1G19DBVRE4, J1 Conn_01x08, J3 Conn_01x08, J4 Conn_01x08, J5 Conn_01x03, J6 Conn_01x08, U1 Am29F040, U2 Am29F040

Commit message: Board routed
Parts:
- added C3: 100nF, Capacitor_SMD:C_0603_1608Metric, F.Cu at (115.3, 83.7)
- C1, C2, R1: moved to B.Cu
- IC1: moved to F.Cu
- moved C2 39.6 mm to (94.4, 92.1)
- moved C1 23.1 mm to (77.8, 94.6), turned to 180 degrees
- moved R1 16.1 mm to (121.5, 74.0), turned to 0 degrees
- moved J1 15.3 mm to (123.2, 88.5), turned to 0 degrees
- moved IC1 14.8 mm to (115.3, 80.8), turned to 180 degrees
- moved J6 14.6 mm to (111.6, 79.5), turned to 180 degrees
- moved J3 8.90 mm to (112.5, 91.5), turned to -90 degrees
- moved J4 8.90 mm to (121.4, 76.5), turned to 90 degrees
- moved J5 3.16 mm to (118.1, 71.8)
Connections:
- net Net-(IC1-~{E}) renamed /CE_SELECT_CONN
- J1 pad 1: /P12 -> /P5
- J1 pad 2: /P11 -> /P6
- J1 pad 3: /P10 -> /P7
- J1 pad 4: /P9 -> /P8
- J1 pad 5: /P8 -> /P9
- J1 pad 6: /P7 -> /P10
- J1 pad 7: /P6 -> /P11
- J1 pad 8: /P5 -> /P12
- J3 pad 1: /P4 -> /P29
- J3 pad 2: /P3 -> /P30
- J3 pad 3: /P2 -> /P31
- J3 pad 4: /P1 -> VCC
- J3 pad 5: VCC -> /P1
- J3 pad 6: /P31 -> /P2
- J3 pad 7: /P30 -> /P3
- J3 pad 8: /P29 -> /P4
- J4 pad 1: /P20 -> /P13
- J4 pad 2: /P19 -> /P14
- J4 pad 3: /P18 -> /P15
- J4 pad 4: /P17 -> GND
- J4 pad 5: GND -> /P17
- J4 pad 6: /P15 -> /P18
- J4 pad 7: /P14 -> /P19
- J4 pad 8: /P13 -> /P20
- J6 pad 1: /P28 -> /P21
- J6 pad 2: /P27 -> /~{CE}
- J6 pad 3: /P26 -> /P23
- J6 pad 4: /P25 -> /P24
- J6 pad 5: /P24 -> /P25
- J6 pad 6: /P23 -> /P26
- J6 pad 7: /~{CE} -> /P27
- J6 pad 8: /P21 -> /P28
- U1 pad 28: /P13 -> /P28
- U1 pad 29: /P14 -> /P29
- U2 pad 28: /P13 -> /P28
- U2 pad 29: /P14 -> /P29
Routing:
- net GND: track 0.00 -> 113.7 mm, vias 0 -> 21
- net VCC: track 0.00 -> 83.0 mm, vias 0 -> 4
- net /P13: track 0.00 -> 53.3 mm, vias 0 -> 4
- net /P14: track 0.00 -> 51.6 mm, vias 0 -> 4
- net /P15: track 0.00 -> 51.2 mm, vias 0 -> 4
- net CE1: track 0.00 -> 51.1 mm, vias 0 -> 2
- net /P17: track 0.00 -> 49.4 mm, vias 0 -> 4
- net /P4: track 0.00 -> 48.0 mm, vias 0 -> 2
- net /P18: track 0.00 -> 47.4 mm, vias 0 -> 4
- net /P3: track 0.00 -> 47.2 mm, vias 0 -> 2
- net /P19: track 0.00 -> 47.1 mm, vias 0 -> 4
- net /P2: track 0.00 -> 45.9 mm, vias 0 -> 2
- net /P1: track 0.00 -> 44.3 mm, vias 0 -> 2
- net /P30: track 0.00 -> 43.6 mm, vias 0 -> 2
- net /P31: track 0.00 -> 43.3 mm, vias 0 -> 2
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- added copper zone on B.Cu, net GND
- added copper zone on F.Cu, net GND
Other:
- board outline removed
