File: DualFlash adapter/dual flash adapter.kicad_sch (KiCad schematic)
At the start: 11 parts, among them IC1 SN74LVC1G19DBVRE4, J1 Conn_01x08, J3 Conn_01x08, J4 Conn_01x08, J5 Conn_01x03, J6 Conn_01x08, U1 Am29F040, U2 Am29F040

Commit message: Board routed
Parts:
- removed J6: Conn_01x08, Connector_PinHeader_1.27mm:PinHeader_1x08_P1.27mm_Vertical, symbol Connector_Generic:Conn_01x08
- added C3: 100nF, Capacitor_SMD:C_0603_1608Metric, symbol Device:C
- added J2: Conn_01x08, Connector_PinHeader_1.27mm:PinHeader_1x08_P1.27mm_Vertical, symbol Connector_Generic:Conn_01x08
Connections:
- net GND: now also C3.2, J2.4 (Pin_4); no longer J4.5 (Pin_5)
- net P1: now also J3.5 (Pin_5); no longer J3.4 (Pin_4)
- net P10: now also J1.6 (Pin_6); no longer J1.3 (Pin_3)
- net P11: now also J1.7 (Pin_7); no longer J1.2 (Pin_2)
- net P12: now also J1.8 (Pin_8); no longer J1.1 (Pin_1)
- net P13: now also J2.1 (Pin_1); no longer J4.8 (Pin_8)
- net P14: now also J2.2 (Pin_2); no longer J4.7 (Pin_7)
- net P15: now also J2.3 (Pin_3); no longer J4.6 (Pin_6)
- net P17: now also J2.5 (Pin_5); no longer J4.4 (Pin_4)
- net P18: now also J2.6 (Pin_6); no longer J4.3 (Pin_3)
- net P19: now also J2.7 (Pin_7); no longer J4.2 (Pin_2)
- net P2: now also J3.6 (Pin_6); no longer J3.3 (Pin_3)
- net P20: now also J2.8 (Pin_8); no longer J4.1 (Pin_1)
- net P21: now also J4.1 (Pin_1)
- net P23: now also J4.3 (Pin_3)
- net P24: now also J4.4 (Pin_4)
- net P25: now also J4.5 (Pin_5)
- net P26: now also J4.6 (Pin_6)
- net P27: now also J4.7 (Pin_7)
- net P28: now also J4.8 (Pin_8)
- net P29: now also J3.1 (Pin_1); no longer J3.8 (Pin_8)
- net P3: now also J3.7 (Pin_7); no longer J3.2 (Pin_2)
- net P30: now also J3.2 (Pin_2); no longer J3.7 (Pin_7)
- net P31: now also J3.3 (Pin_3); no longer J3.6 (Pin_6)
- net P4: now also J3.8 (Pin_8); no longer J3.1 (Pin_1)
- net P5: now also J1.1 (Pin_1); no longer J1.8 (Pin_8)
- net P6: now also J1.2 (Pin_2); no longer J1.7 (Pin_7)
- net P7: now also J1.3 (Pin_3); no longer J1.6 (Pin_6)
- net P8: now also J1.4 (Pin_4); no longer J1.5 (Pin_5)
- net P9: now also J1.5 (Pin_5); no longer J1.4 (Pin_4)
- net VCC: now also J3.4 (Pin_4), C3.1; no longer J3.5 (Pin_5)
- net ~{CE}: now also J4.2 (Pin_2)
- net CE_SELECT_CONN: now reaches IC1.3 (~{E}), J5.2 (Pin_2), R1.2
Other:
- moved on the sheet: J5

Commit message: Repo update
Parts:
- removed J2: Conn_01x08, Connector_PinHeader_1.27mm:PinHeader_1x08_P1.27mm_Vertical, symbol Connector_Generic:Conn_01x08
- added J6: Conn_01x08, Connector_PinHeader_1.27mm:PinHeader_1x08_P1.27mm_Vertical, symbol Connector_Generic:Conn_01x08
Connections:
- net GND: now also J4.4 (Pin_4)
- net P13: now also J4.1 (Pin_1)
- net P14: now also J4.2 (Pin_2)
- net P15: now also J4.3 (Pin_3)
- net P17: now also J4.5 (Pin_5)
- net P18: now also J4.6 (Pin_6)
- net P19: now also J4.7 (Pin_7)
- net P20: now also J4.8 (Pin_8)
- net P21: now also J6.1 (Pin_1); no longer J4.1 (Pin_1)
- net P23: now also J6.3 (Pin_3); no longer J4.3 (Pin_3)
- net P24: now also J6.4 (Pin_4); no longer J4.4 (Pin_4)
- net P25: now also J6.5 (Pin_5); no longer J4.5 (Pin_5)
- net P26: now also J6.6 (Pin_6); no longer J4.6 (Pin_6)
- net P27: now also J6.7 (Pin_7); no longer J4.7 (Pin_7)
- net P28: now also J6.8 (Pin_8); no longer J4.8 (Pin_8)
- net ~{CE}: now also J6.2 (Pin_2); no longer J4.2 (Pin_2)
