File: ESB0100D City-120 mainboard/mow_motor_driver.kicad_sch (KiCad schematic)
At the start: 15 parts, among them J1 Conn_01x02, Q1 SPB18P06P, Q2 IRFZ44N, Q3 NMOS, U3 LM393

Commit message: Daily save
Parts:
- added R22: 10, symbol Device:R
- added RN2: 330, symbol Device:R_Pack04
- added U7: 74153, symbol 74xx_IEEE:74153
- renumbered C2 to C6, J1 to J2, Q3 to Q4, Q1 to Q5, Q2 to Q6, R11 to R28
Connections:
- net at C6.2, Q6.3 (S), R12.1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: now also R14.1
- net at Q6.2 (G), R14.2: now also C6.1, R15.2, R22.2
- new net: RN2.8 (R1.2), U7.14 (A)
- new net: RN2.7 (R2.2), U7.2 (B)
- new net: RN2.6 (R3.2), U7.3 (I3a)
- new net: RN2.5 (R4.2), U7.4 (I2a)
- new net: R22.1, U7.7 (Qa)
- new net MOW_153_MUXES_B: RN2.2 (R2.1)
- new net MOW_153_MUXES_I2A: RN2.4 (R4.1)
- new net MOW_153_MUXES_I3A: RN2.3 (R3.1)
- new net MOW_153_MUX_3_A: RN2.1 (R1.1)
Other:
- moved on the sheet: C3, C4, C6, J2, Q4, Q5, Q6, R12, R13, R15, R16, R17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

Commit message: Repo update
Parts:
- renumbered C6 to C?, J2 to J?, Q4 to Q?, Q6 to Q?, Q5 to Q?, R22 to R?, R28 to R?, RN2 to RN?, U7 to U?
Changed lines of the file:
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@@
 (kicad_sch
-	(version 20231120)
+	(version 20250114)
 	(generator "eeschema")
-	(generator_version "8.0")
+	(generator_version "9.0")
 	(paper "A4")
 	(junction
@@
 	(wire
 		(pts
-			(xy 151.765 135.89) (xy 153.67 135.89)
-		)
-		(stroke
-			(width 0)
-			(type default)
-		)
-	)
-	(wire
-		(pts
 			(xy 173.355 93.345) (xy 173.355 87.63)
 		)
@@
 	(wire
 		(pts
-			(xy 151.765 135.255) (xy 131.445 135.255)
+			(xy 131.445 135.255) (xy 153.67 135.255)
 		)
 		(stroke
@@
 	(wire
 		(pts
-			(xy 153.67 74.93) (xy 153.67 135.89)
+			(xy 153.67 74.93) (xy 153.67 135.255)
 		)
 		(stroke
@@
 		(pts
 			(xy 139.065 74.93) (xy 139.065 76.835)
-		)
-		(stroke
-			(width 0)
-			(type default)
-		)
-	)
-	(wire
-		(pts
-			(xy 151.765 135.89) (xy 151.765 135.255)
 		)
 		(stroke
@@
 		(dnp no)
 		(fields_autoplaced yes)
-		(property "Reference" "J2"
+		(property "Reference" "J?"
 			(at 200.66 73.0249 0)
 			(effects
@@
 		(instances
 			(project "ESB0100D City-120 mainboard"
+				(path "/1b7d23ce-0357-4769-ae9f-ddb2c39b8a27/62c08ad4-e951-41c5-8870-3408b773ffe0"
+					(reference "J?")
+					(unit 1)
+				)
 				(path "/1b7d23ce-0357-4769-ae9f-ddb2c39b8a27/ce624f23-37bc-4c79-877d-7124c0db9091"
 					(reference "J2")
@@
 		(dnp no)
 		(fields_autoplaced yes)
-		(property "Reference" "Q4"
+		(property "Reference" "Q?"
 			(at 52.07 38.0999 0)
 			(effects
@@
 		(instances
 			(project "ESB0100D City-120 mainboard"
+				(path "/1b7d23ce-0357-4769-ae9f-ddb2c39b8a27/62c08ad4-e951-41c5-8870-3408b773ffe0"
+					(reference "Q?")
+					(unit 1)
+				)
 				(path "/1b7d23ce-0357-4769-ae9f-ddb2c39b8a27/ce624f23-37bc-4c79-877d-7124c0db9091"
 					(reference "Q4")
@@
 		(dnp no)
 		(fields_autoplaced yes)
-		(property "Reference" "U7"
+		(property "Reference" "U?"
 			(at 96.8091 100.33 0)
 			(effects
@@
 		(instances
 			(project "ESB0100D City-120 mainboard"
+				(path "/1b7d23ce-0357-4769-ae9f-ddb2c39b8a27/62c08ad4-e951-41c5-8870-3408b773ffe0"
+					(reference "U?")
+					(unit 1)
+				)
 				(path "/1b7d23ce-0357-4769-ae9f-ddb2c39b8a27/ce624f23-37bc-4c79-877d-7124c0db9091"
 					(reference "U7")
@@
 		(dnp no)
 		(fields_autoplaced yes)
-		(property "Reference" "Q6"
+		(property "Reference" "Q?"
 			(at 176.53 73.6599 0)
 			(effects
@@
 		(instances
 			(project "ESB0100D City-120 mainboard"
+				(path "/1b7d23ce-0357-4769-ae9f-ddb2c39b8a27/62c08ad4-e951-41c5-8870-3408b773ffe0"
+					(reference "Q?")
+					(unit 1)
+				)
 				(path "/1b7d23ce-0357-4769-ae9f-ddb2c39b8a27/ce624f23-37bc-4c79-877d-7124c0db9091"
 					(reference "Q6")
@@
 		(dnp no)
 		(fields_autoplaced yes)
-		(property "Reference" "R22"
+		(property "Reference" "R?"
 			(at 127.635 129.54 90)
 			(effects
@@
 		(instances
 			(project "ESB0100D City-120 mainboard"
+				(path "/1b7d23ce-0357-4769-ae9f-ddb2c39b8a27/62c08ad4-e951-41c5-8870-3408b773ffe0"
+					(reference "R?")
+					(unit 1)
+				)
 				(path "/1b7d23ce-0357-4769-ae9f-ddb2c39b8a27/ce624f23-37bc-4c79-877d-7124c0db9091"
 					(reference "R22")
@@
 		(dnp no)
 		(fields_autoplaced yes)
-		(property "Reference" "RN2"
+		(property "Reference" "RN?"
 			(at 50.165 104.14 90)
 			(effects
@@
 		(instances
 			(project "ESB0100D City-120 mainboard"
+				(path "/1b7d23ce-0357-4769-ae9f-ddb2c39b8a27/62c08ad4-e951-41c5-8870-3408b773ffe0"
+					(reference "RN?")
+					(unit 1)
+				)
 				(path "/1b7d23ce-0357-4769-ae9f-ddb2c39b8a27/ce624f23-37bc-4c79-877d-7124c0db9091"
 					(reference "RN2")
@@
 		(dnp no)
 		(fields_autoplaced yes)
-		(property "Reference" "Q5"
+		(property "Reference" "Q?"
 			(at 176.53 57.7849 0)
 			(effects
@@
 		(instances
 			(project "ESB0100D City-120 mainboard"
+				(path "/1b7d23ce-0357-4769-ae9f-ddb2c39b8a27/62c08ad4-e951-41c5-8870-3408b773ffe0"
+					(reference "Q?")
+					(unit 1)
+				)
 				(path "/1b7d23ce-0357-4769-ae9f-ddb2c39b8a27/ce624f23-37bc-4c79-877d-7124c0db9091"
 					(reference "Q5")
@@
 		(dnp no)
 		(fields_autoplaced yes)
-		(property "Reference" "#PWR26"
+		(property "Reference" "#PWR?"
 			(at 48.26 61.595 0)
 			(effects
@@
 		(instances
 			(project "ESB0100D City-120 mainboard"
+				(path "/1b7d23ce-0357-4769-ae9f-ddb2c39b8a27/62c08ad4-e951-41c5-8870-3408b773ffe0"
+					(reference "#PWR?")
+					(unit 1)
+				)
 				(path "/1b7d23ce-0357-4769-ae9f-ddb2c39b8a27/ce624f23-37bc-4c79-877d-7124c0db9091"
 					(reference "#PWR26")
@@
 		(dnp no)
 		(fields_autoplaced yes)
-		(property "Reference" "C6"
+		(property "Reference" "C?"
 			(at 142.24 79.3749 0)
 			(effects
@@
 		(instances
 			(project "ESB0100D City-120 mainboard"
+				(path "/1b7d23ce-0357-4769-ae9f-ddb2c39b8a27/62c08ad4-e951-41c5-8870-3408b773ffe0"
+					(reference "C?")
+					(unit 1)
+				)
 				(path "/1b7d23ce-0357-4769-ae9f-ddb2c39b8a27/ce624f23-37bc-4c79-877d-7124c0db9091"
 					(reference "C6")
@@
 		(dnp no)
 		(fields_autoplaced yes)
-		(property "Reference" "#PWR27"
+		(property "Reference" "#PWR?"
 			(at 165.1 111.125 0)
 			(effects
@@
 		(instances
 			(project "ESB0100D City-120 mainboard"
+				(path "/1b7d23ce-0357-4769-ae9f-ddb2c39b8a27/62c08ad4-e951-41c5-8870-3408b773ffe0"
+					(reference "#PWR?")
+					(unit 1)
+				)
 				(path "/1b7d23ce-0357-4769-ae9f-ddb2c39b8a27/ce624f23-37bc-4c79-877d-7124c0db9091"
 					(reference "#PWR27")
@@
 		(dnp no)
 		(fields_autoplaced yes)
-		(property "Reference" "R28"
+		(property "Reference" "R?"
 			(at 184.785 95.8849 0)
 			(effects
@@
 		(instances
 			(project "ESB0100D City-120 mainboard"
+				(path "/1b7d23ce-0357-4769-ae9f-ddb2c39b8a27/62c08ad4-e951-41c5-8870-3408b773ffe0"
+					(reference "R?")
+					(unit 1)
+				)
 				(path "/1b7d23ce-0357-4769-ae9f-ddb2c39b8a27/ce624f23-37bc-4c79-877d-7124c0db9091"
 					(reference "R28")
